Commit message: fixed the chasis dimentions

File: description/robot_core.xacro (robot description, xacro)
@@ -22,7 +22,7 @@
     <link name="chassis">
         <visual>
-            <origin xyz="0.127 0 0"/>
+            <origin xyz="0.128 0 0"/>
             <geometry>
-                <box size="0.26035 0.1524 0.0381"/>
+                <box size="0.256 0.15 0.035"/>
             </geometry>
             <material name="white"/>
@@ -31,16 +31,19 @@
             <origin xyz="0 0 0"/>
             <geometry>
-                <box size="0.254 0.1524 0.15"/>
+                <box size="0.256 0.15 0.035"/>
             </geometry>
         </collision>
         <xacro:inertial_box mass="0.5" x="0.254" y="0.1524" z="0.15">
-            <origin xyz="0 0 0" rpy="0 0 0"/>
+            <origin xyz="0.128 0 0" rpy="0 0 0"/>
         </xacro:inertial_box>
     </link>
+    <gazebo reference="chassis">
+        <material>Gazebo/White</material>
+    </gazebo>
     <!-- LEFT FRONT WHEEL LINK -->
     <joint name="left_front_wheel_joint" type="continuous">
         <parent link="base_link"/>
         <child link="left_front_wheel"/>
-        <origin xyz="0.0762 0.0762 0" rpy="-${pi/2} 0 0" />
+        <origin xyz="0.06 0.065 0" rpy="-${pi/2} 0 0" />
         <axis xyz="0 0 1"/>
     </joint>
@@ -48,5 +51,5 @@
         <visual>
             <geometry>
-                <cylinder radius="0.0381" length="0.04"/>
+                <cylinder radius="0.035" length="0.025"/>
             </geometry>
             <material name="blue"/>
@@ -54,16 +57,19 @@
         <collision>
             <geometry>
-                <cylinder radius="0.0381" length="0.04"/>
+                <cylinder radius="0.035" length="0.025"/>
             </geometry>
         </collision>
-        <xacro:inertial_cylinder mass="0.1" length="0.04" radius="0.0381">
+        <xacro:inertial_cylinder mass="0.1" length="0.025" radius="0.035">
             <origin xyz="0 0 0" rpy="1.5708 0 0"/>
         </xacro:inertial_cylinder>
     </link>
+    <gazebo reference="left_front_wheel">
+        <material>Gazebo/Blue</material>
+    </gazebo>
     <!-- RIGHT FRONT WHEEL LINK -->
     <joint name="right_front_wheel_joint" type="continuous">
         <parent link="base_link"/>
         <child link="right_front_wheel"/>
-        <origin xyz="0.0762 -0.0762 0" rpy="${pi/2} 0 0" />
+        <origin xyz="0.06 -0.065 0" rpy="${pi/2} 0 0" />
         <axis xyz="0 0 -1"/>
     </joint>
@@ -71,5 +77,5 @@
         <visual>
             <geometry>
-                <cylinder radius="0.0381" length="0.04"/>
+                <cylinder radius="0.035" length="0.025"/>
             </geometry>
             <material name="blue"/>
@@ -77,16 +83,19 @@
         <collision>
             <geometry>
-                <cylinder radius="0.0381" length="0.04"/>
+                <cylinder radius="0.035" length="0.025"/>
             </geometry>
         </collision>
-        <xacro:inertial_cylinder mass="0.1" length="0.04" radius="0.0381">
+        <xacro:inertial_cylinder mass="0.1" length="0.025" radius="0.035">
             <origin xyz="0 0 0" rpy="1.5708 0 0"/>
         </xacro:inertial_cylinder>
     </link>
+    <gazebo reference="right_front_wheel">
+        <material>Gazebo/Blue</material>
+    </gazebo>
     <!-- LEFT REAR WHEEL LINK -->
     <joint name="left_rear_wheel_joint" type="continuous">
         <parent link="base_link"/>
         <child link="left_rear_wheel"/>
-        <origin xyz="-0.0762 0.0762 0" rpy="-${pi/2} 0 0" />
+        <origin xyz="-0.06 0.065 0" rpy="-${pi/2} 0 0" />
         <axis xyz="0 0 1"/>
     </joint>
@@ -94,5 +103,5 @@
         <visual>
             <geometry>
-                <cylinder radius="0.0381" length="0.04"/>
+                <cylinder radius="0.035" length="0.025"/>
             </geometry>
             <material name="blue"/>
@@ -100,16 +109,19 @@
         <collision>
             <geometry>
-                <cylinder radius="0.0381" length="0.04"/>
+                <cylinder radius="0.035" length="0.025"/>
             </geometry>
         </collision>
-        <xacro:inertial_cylinder mass="0.1" length="0.04" radius="0.0381">
+        <xacro:inertial_cylinder mass="0.1" length="0.025" radius="0.035">
             <origin xyz="0 0 0" rpy="1.5708 0 0"/>
         </xacro:inertial_cylinder>
     </link>
+    <gazebo reference="left_rear_wheel">
+        <material>Gazebo/Blue</material>
+    </gazebo>
     <!-- RIGHT REAR WHEEL LINK -->
     <joint name="right_rear_wheel_joint" type="continuous">
         <parent link="base_link"/>
         <child link="right_rear_wheel"/>
-        <origin xyz="-0.0762 -0.0762 0" rpy="${pi/2} 0 0" />
+        <origin xyz="-0.06 -0.065 0" rpy="${pi/2} 0 0" />
         <axis xyz="0 0 -1"/>
     </joint>
@@ -117,5 +129,5 @@
         <visual>
             <geometry>
-                <cylinder radius="0.0381" length="0.04"/>
+                <cylinder radius="0.035" length="0.025"/>
             </geometry>
             <material name="blue"/>
@@ -123,10 +135,13 @@
         <collision>
             <geometry>
-                <cylinder radius="0.0381" length="0.04"/>
+                <cylinder radius="0.035" length="0.025"/>
             </geometry>
         </collision>
-        <xacro:inertial_cylinder mass="0.1" length="0.04" radius="0.0381">
+        <xacro:inertial_cylinder mass="0.1" length="0.025" radius="0.035">
             <origin xyz="0 0 0" rpy="1.5708 0 0"/>
         </xacro:inertial_cylinder>
     </link>
+    <gazebo reference="right_rear_wheel">
+        <material>Gazebo/Blue</material>
+    </gazebo>
 </robot>
