Commit message: Updated skid steer NOW WORKINGgit status(Tue Nov 28 04:08:57 AM EST 2023)

File: description/gazebo_control.xacro (robot description, xacro)
@@ -2,27 +2,26 @@
 <robot xmlns:xacro="http://www.ros.org/wiki/xacro">
     <gazebo>
-        <plugin name="skid_steer_drive_controller" filename="libgazebo_ros_skid_steer_drive.so">
-            <updateRate>10.0</updateRate>
-            <robotNamespace>/my_bot</robotNamespace>
-            <leftFrontJoint>left_front_wheel_joint</leftFrontJoint>
-            <rightFrontJoint>right_front_wheel_joint</rightFrontJoint>
-            <leftRearJoint>left_rear_wheel_joint</leftRearJoint>
-            <rightRearJoint>right_rear_wheel_joint</rightRearJoint>
-            <wheelSeparation>0.4</wheelSeparation>
-            <wheelDiameter>0.2</wheelDiameter>
-            <robotBaseFrame>base_link</robotBaseFrame>
-            <torque>10</torque>
-            <topicName>cmd_vel</topicName>
-            <odometryTopic>odom</odometryTopic>
-            <odometryFrame>odom</odometryFrame>
-            <commandTopic>cmd_vel</commandTopic>
-            <topic_name_twist>cmd_vel</topic_name_twist>
-            <topic_name_odometry>odom</topic_name_odometry>
-            <topic_name_joint>joint</topic_name_joint>
-            <broadcastTF>true</broadcastTF>
-            <covariance_x>0.0001</covariance_x>
-            <covariance_y>0.0001</covariance_y>
-            <covariance_yaw>0.01</covariance_yaw>
+        <plugin name='diff_drive' filename='libgazebo_ros_diff_drive.so'>
+        <num_wheel_pairs>2</num_wheel_pairs>
+            <!-- Wheel Information -->
+        <left_joint>left_front_wheel_joint</left_joint>
+        <left_joint>left_rear_wheel_joint</left_joint>
+        <!-- Right Wheel Joints -->
+        <right_joint>right_front_wheel_joint</right_joint>
+        <right_joint>right_rear_wheel_joint</right_joint>
+        <!-- Wheel Separation and Diameter -->
+        <wheel_separation>0.2</wheel_separation> <!-- Adjust as needed -->
+        <wheel_diameter>0.07</wheel_diameter> <!-- Adjust as needed -->
+        <!-- Wheel Torque and Acceleration Limits -->
+        <max_wheel_torque>20</max_wheel_torque>
+        <max_wheel_acceleration>10.0</max_wheel_acceleration>
+        <!-- Odometry and Transform Frames -->
+        <odometry_frame>odom</odometry_frame>
+        <robot_base_frame>base_link</robot_base_frame>
+        <!-- Additional Options -->
+        <publish_odom>true</publish_odom>
+        <publish_odom_tf>true</publish_odom_tf>
+        <publish_wheel_tf>true</publish_wheel_tf>
         </plugin>
-     </gazebo>
+    </gazebo>
 </robot>

File: description/robot_core.xacro (robot description, xacro)
@@ -47,4 +47,5 @@
         <origin xyz="0.06 0.065 0" rpy="-${pi/2} 0 0" />
         <axis xyz="0 0 1"/>
+        <limit lower="-3.1416" upper="3.1416" effort="10" velocity="10"/>
     </joint>
     <link name="left_front_wheel">
@@ -73,4 +74,5 @@
         <origin xyz="0.06 -0.065 0" rpy="${pi/2} 0 0" />
         <axis xyz="0 0 -1"/>
+        <limit lower="-3.1416" upper="3.1416" effort="10" velocity="10"/>
     </joint>
     <link name="right_front_wheel">
@@ -99,4 +101,5 @@
         <origin xyz="-0.06 0.065 0" rpy="-${pi/2} 0 0" />
         <axis xyz="0 0 1"/>
+        <limit lower="-3.1416" upper="3.1416" effort="10" velocity="10"/>
     </joint>
     <link name="left_rear_wheel">
@@ -125,4 +128,5 @@
         <origin xyz="-0.06 -0.065 0" rpy="${pi/2} 0 0" />
         <axis xyz="0 0 -1"/>
+        <limit lower="-3.1416" upper="3.1416" effort="10" velocity="10"/>
     </joint>
     <link name="right_rear_wheel">
